Commit message: feat: 完善 Aloha 底盘仿真控制功能
- 修复 URDF 升降关节偏移问题：在 visualizer.py 中补偿 0.45m 基础高度
- 实现完整的三自由度底盘控制：前进/后退、左右平移、转向旋转
- 修正仿真运动学逻辑：车身坐标系速度正确转换到世界坐标系
- 优化控制参数：线速度 1.0 m/s，角速度 1.0 deg/s
- 分离仿真与真机数据流：仿真直接使用 vx/vy/vtheta，真机经过 wheels 逆解
- 翻译配置文件注释：config.py 和 visualizer.py 全部中文化

File: URDF/aloha/Aloha.urdf (robot description, URDF)
Before this commit: robot Aloha, 19 links, 18 joints
Joints:
- joint vertical_move: origin xyz=-0.001045 -0.067891 0.064 rpy=0 0 0 -> xyz=-0.001045 -0.067891 0 rpy=0 0 0
