Commit message: 加了限位，待测试

File: URDF/aider/urdf/aider_pro.SLDASM.urdf (robot description, URDF)
Before this commit: robot aider_pro.SLDASM, 25 links, 24 joints
Joints:
- joint head_Link: limit lower=0 upper=0 effort=0 velocity=0 -> lower=-1.0472 upper=1.0472 effort=0 velocity=0
- joint head_Link2: limit lower=0 upper=0 effort=0 velocity=0 -> lower=-0.5236 upper=0.7854 effort=0 velocity=0
- joint left_arm1: limit lower=0 upper=0 effort=0 velocity=0 -> lower=-1.5708 upper=1.5708 effort=0 velocity=0
- joint left_arm2: limit lower=0 upper=0 effort=0 velocity=0 -> lower=-2.618 upper=0.5236 effort=0 velocity=0
- joint left_arm3: limit lower=0 upper=0 effort=0 velocity=0 -> lower=-2.618 upper=0.5236 effort=0 velocity=0
- joint left_arm4: limit lower=0 upper=0 effort=0 velocity=0 -> lower=-1.5708 upper=1.5708 effort=0 velocity=0
- joint left_arm5: limit lower=0 upper=0 effort=0 velocity=0 -> lower=-0.7854 upper=0.7854 effort=0 velocity=0
- joint left_arm6: limit lower=0 upper=0 effort=0 velocity=0 -> lower=-1.2217 upper=1.2217 effort=0 velocity=0
- joint left_arm7: limit lower=0 upper=0 effort=0 velocity=0 -> lower=-0.7854 upper=0.7854 effort=0 velocity=0
- joint left_arm8: limit lower=0 upper=0 effort=0 velocity=0 -> lower=-1.5708 upper=0 effort=0 velocity=0
- joint lift_Link: limit lower=0 upper=0 effort=0 velocity=0 -> lower=0 upper=0.5 effort=0 velocity=0
- joint right_arm1: limit lower=0 upper=0 effort=0 velocity=0 -> lower=-1.5708 upper=1.5708 effort=0 velocity=0
- joint right_arm2: limit lower=0 upper=0 effort=0 velocity=0 -> lower=-2.618 upper=0.5236 effort=0 velocity=0
- joint right_arm3: limit lower=0 upper=0 effort=0 velocity=0 -> lower=-2.618 upper=0.5236 effort=0 velocity=0
- joint right_arm4: limit lower=0 upper=0 effort=0 velocity=0 -> lower=-1.5708 upper=1.5708 effort=0 velocity=0
- joint right_arm5: limit lower=0 upper=0 effort=0 velocity=0 -> lower=-0.7854 upper=0.7854 effort=0 velocity=0
- joint right_arm6: limit lower=0 upper=0 effort=0 velocity=0 -> lower=-1.2217 upper=1.2217 effort=0 velocity=0
- joint right_arm7: limit lower=0 upper=0 effort=0 velocity=0 -> lower=-0.7854 upper=0.7854 effort=0 velocity=0
- joint right_arm8: limit lower=0 upper=0 effort=0 velocity=0 -> lower=-1.5708 upper=0 effort=0 velocity=0
- joint waist_Link: limit lower=0 upper=0 effort=0 velocity=0 -> lower=-1.5708 upper=1.5708 effort=0 velocity=0

Commit message: ik ok拉

File: URDF/aider/urdf/aider_pro.SLDASM.urdf (robot description, URDF)
Before this commit: robot aider_pro.SLDASM, 25 links, 24 joints
Joints:
- joint head_Link: limit lower=-1.0472 upper=1.0472 effort=0 velocity=0 -> lower=-1.04719755 upper=1.04719755 effort=0 velocity=0
- joint head_Link2: limit lower=-0.5236 upper=0.7854 effort=0 velocity=0 -> lower=-0.52359878 upper=0.78539816 effort=0 velocity=0
- joint left_arm1: limit lower=-1.5708 upper=1.5708 effort=0 velocity=0 -> lower=-2.35619449 upper=2.35619449 effort=0 velocity=0
- joint left_arm2: limit lower=-2.618 upper=0.5236 effort=0 velocity=0 -> lower=-2.61799388 upper=1.57079633 effort=0 velocity=0
- joint left_arm3: limit lower=-2.618 upper=0.5236 effort=0 velocity=0 -> lower=-1.57079633 upper=1.57079633 effort=0 velocity=0
- joint left_arm4: limit lower=-1.5708 upper=1.5708 effort=0 velocity=0 -> lower=0.00000000 upper=2.35619449 effort=0 velocity=0
- joint left_arm5: limit lower=-0.7854 upper=0.7854 effort=0 velocity=0 -> lower=-1.57079633 upper=1.57079633 effort=0 velocity=0
- joint left_arm6: limit lower=-1.2217 upper=1.2217 effort=0 velocity=0 -> lower=-1.57079633 upper=1.57079633 effort=0 velocity=0
- joint left_arm7: limit lower=-0.7854 upper=0.7854 effort=0 velocity=0 -> lower=-1.57079633 upper=1.57079633 effort=0 velocity=0
- joint left_arm8: limit lower=-1.5708 upper=0 effort=0 velocity=0 -> lower=-1.57079633 upper=0.00000000 effort=0 velocity=0
- joint lift_Link: limit lower=0 upper=0.5 effort=0 velocity=0 -> lower=0.00000000 upper=0.50000000 effort=0 velocity=0
- joint right_arm1: limit lower=-1.5708 upper=1.5708 effort=0 velocity=0 -> lower=-2.35619449 upper=2.35619449 effort=0 velocity=0
- joint right_arm2: limit lower=-2.618 upper=0.5236 effort=0 velocity=0 -> lower=-2.61799388 upper=1.57079633 effort=0 velocity=0
- joint right_arm3: limit lower=-2.618 upper=0.5236 effort=0 velocity=0 -> lower=-1.57079633 upper=1.57079633 effort=0 velocity=0
- joint right_arm4: limit lower=-1.5708 upper=1.5708 effort=0 velocity=0 -> lower=-2.35619449 upper=0.00000000 effort=0 velocity=0
- joint right_arm5: limit lower=-0.7854 upper=0.7854 effort=0 velocity=0 -> lower=-1.57079633 upper=1.57079633 effort=0 velocity=0
- joint right_arm6: limit lower=-1.2217 upper=1.2217 effort=0 velocity=0 -> lower=-1.57079633 upper=1.57079633 effort=0 velocity=0
- joint right_arm7: limit lower=-0.7854 upper=0.7854 effort=0 velocity=0 -> lower=-1.57079633 upper=1.57079633 effort=0 velocity=0
- joint right_arm8: limit lower=-1.5708 upper=0 effort=0 velocity=0 -> lower=-1.57079633 upper=0.00000000 effort=0 velocity=0
- joint waist_Link: limit lower=-1.5708 upper=1.5708 effort=0 velocity=0 -> lower=-1.57079633 upper=1.57079633 effort=0 velocity=0
