Commit message: 导入新URDF

File: URDF/aider/urdf/aider_pro.SLDASM.urdf (robot description, URDF)
Before this commit: robot aider_pro.SLDASM, 25 links, 24 joints
Links:
- added link left_hand_tcp, mass 0.000144; collision mesh filename=package://aider_pro.SLDASM/meshes/left_hand_tcp.STL; visual mesh filename=package://aider_pro.SLDASM/meshes/left_hand_tcp.STL
- added link right_hand_tcp, mass 0.000144; collision mesh filename=package://aider_pro.SLDASM/meshes/right_hand_tcp.STL; visual mesh filename=package://aider_pro.SLDASM/meshes/right_hand_tcp.STL
- link base_link: mass 10.0947181370065 -> 1.8672299751897
- link head_Link: mass 0.026573709748435 -> 0.0401514926582811
- link head_Link2: mass 0.0191222199222675 -> 0.189625426643452
- link left_arm1: mass 0.268295377998009 -> 0.2771689234867
- link left_arm2: mass 0.163192915901943 -> 0.173551520246761
- link left_arm3: mass 0.156973074825494 -> 0.162415224100578
- link left_arm4: mass 0.0544493684812528 -> 0.061262551263452
- link left_arm5: mass 0.0481301580835354 -> 0.0503857298730898
- link left_arm6: mass 0.0604588482328481 -> 0.0471985933288053
- link left_arm7: mass 0.0537494297745682 -> 0.103857648360567
- link left_arm8: mass 0.0215255368998184 -> 0.0398761874096987
- link lift_Link: mass 0.460714901304408 -> 0.590735662767956
- link right_arm1: mass 0.26396103273574 -> 0.27717
- link right_arm2: mass 0.163192877536271 -> 0.210693834825324
- link right_arm3: mass 0.156972943684637 -> 0.16242
- link right_arm4: mass 0.0544493322914559 -> 0.0612625148219103
- link right_arm5: mass 0.0481301284115415 -> 0.050386
- link right_arm6: mass 0.0328286145276286 -> 0.047198
- link right_arm7: mass 0.0537494230519702 -> 0.103857535053998
- link right_arm8: mass 0.0215255368998188 -> 0.039876
- link waist_Link: mass 0.771104035624796 -> 1.90391027149609
- link whel_Link1: mass 0.313871677020867 -> 0.286092916963456
- link whel_Link2: mass 0.313871844080469 -> 0.286092750982276
- link whel_Link3: mass 0.313871677020866 -> 0.286092916963456
- link whel_Link4: mass 0.313871844080469 -> None
Joints:
- added joint left_hand_tcp: type fixed, parent left_arm8, child left_hand_tcp, origin xyz=-0.0285425250176357 0.12828023583548 -0.0210756042379271 rpy=0 0 0, axis 0 0 0
- added joint right_hand_tcp: type fixed, parent right_arm8, child right_hand_tcp, origin xyz=0.0171000000000001 0.12828023583548 -0.0210756042379271 rpy=0 0 0, axis 0 0 0
- joint head_Link: limit lower=-1.04719755 upper=1.04719755 effort=0 velocity=0 -> lower=0 upper=0 effort=0 velocity=0; origin xyz=-0.00190000759412484 0.0149162354005041 0.380700000000015 rpy=0 0 0 -> xyz=0 -0.163916235400507 0.448200000000012 rpy=0 0 0
- joint head_Link2: limit lower=-0.52359878 upper=0.78539816 effort=0 velocity=0 -> lower=0 upper=0 effort=0 velocity=0; origin xyz=-0.0182000000001125 -0.0153487797565757 0.0134617039078002 rpy=0 0 0 -> xyz=-0.0183049377506555 -0.0130000000000431 0.0225999999999615 rpy=0 0 0
- joint left_arm1: limit lower=-2.35619449 upper=2.35619449 effort=0 velocity=0 -> lower=0 upper=0 effort=0 velocity=0; origin xyz=0.0897100000000015 1.40841572892347E-05 0.265000000000003 rpy=0 0 0 -> xyz=0.105510000000001 -0.148985915842714 0.3225 rpy=0 0 0
- joint left_arm2: axis 0 -1 0 -> 0 1 0; limit lower=-2.61799388 upper=1.57079633 effort=0 velocity=0 -> lower=0 upper=0 effort=0 velocity=0; origin xyz=0.048 -0.0245 0 rpy=0 0 0 -> xyz=0.0420000000000001 -0.0399999999999999 0 rpy=0 0 0
- joint left_arm3: axis 0 0 -1 -> 0 0 1; limit lower=-1.57079633 upper=1.57079633 effort=0 velocity=0 -> lower=0 upper=0 effort=0 velocity=0; origin xyz=0 0.0264999806952237 -0.1184 rpy=0 0 0 -> xyz=0 0.0399999806952274 -0.133399999999999 rpy=0 0 0
- joint left_arm4: axis -1 0 0 -> 1 0 0; limit lower=0.00000000 upper=2.35619449 effort=0 velocity=0 -> lower=0 upper=0 effort=0 velocity=0; origin xyz=-0.0154000000000001 0 -0.123 rpy=0 0 0 -> xyz=-0.0244 0 -0.115 rpy=0 0 0
- joint left_arm5: axis 0 0 -1 -> 0 0 1; limit lower=-1.57079633 upper=1.57079633 effort=0 velocity=0 -> lower=0 upper=0 effort=0 velocity=0; origin xyz=0.0209999999999991 0 -0.102074645752273 rpy=0 0 0 -> xyz=0.032 0 -0.12 rpy=0 0 0
- joint left_arm6: axis -1 0 0 -> 1 0 0; limit lower=-1.57079633 upper=1.57079633 effort=0 velocity=0 -> lower=0 upper=0 effort=0 velocity=0; origin xyz=-0.0114899959967967 0 -0.111282746643053 rpy=0 0 0 -> xyz=-0.018 0 -0.10136 rpy=0 0 0
- joint left_arm7: axis 0 -1 0 -> 0 1 0; limit lower=-1.57079633 upper=1.57079633 effort=0 velocity=0 -> lower=0 upper=0 effort=0 velocity=0; origin xyz=0.0214170897275938 -0.0219000000001115 -0.0583391608133423 rpy=0 0 0 -> xyz=0.0275 -0.02965 -0.05999 rpy=0 0 0
- joint left_arm8: axis -1 0 0 -> 1 0 0; limit lower=-1.57079633 upper=0.00000000 effort=0 velocity=0 -> lower=0 upper=0 effort=0 velocity=0; origin xyz=-0.0219000000001126 0.00615122024342424 -0.0373617039078 rpy=0 0 0 -> xyz=0.028543 0.025417 -0.065349 rpy=0 0 0
- joint lift_Link: limit lower=0.00000000 upper=0.50000000 effort=0 velocity=0 -> lower=0 upper=0 effort=0 velocity=0; origin xyz=0 -0.0929999999999998 1.405 rpy=0 0 0 -> xyz=0 -0.0930000000000004 0.577289106240448 rpy=0 0 0
- joint right_arm1: limit lower=-2.35619449 upper=2.35619449 effort=0 velocity=0 -> lower=0 upper=0 effort=0 velocity=0; origin xyz=-0.0620099999999999 1.4084157292038E-05 0.265000000000001 rpy=0 0 0 -> xyz=-0.0650100000000005 -0.14898591584271 0.322499999999999 rpy=0 0 0
- joint right_arm2: limit lower=-2.61799388 upper=1.57079633 effort=0 velocity=0 -> lower=0 upper=0 effort=0 velocity=0; origin xyz=-0.0795 -0.0205000000000028 0 rpy=0 0 0 -> xyz=-0.0825 -0.0205 0 rpy=0 0 0
- joint right_arm3: limit lower=-1.57079633 upper=1.57079633 effort=0 velocity=0 -> lower=0 upper=0 effort=0 velocity=0; origin xyz=0 0.0224999806952237 -0.1184 rpy=0 0 0 -> xyz=0 0.0204999806952246 -0.1204 rpy=0 0 0
- joint right_arm4: limit lower=-2.35619449 upper=0.00000000 effort=0 velocity=0 -> lower=0 upper=0 effort=0 velocity=0; origin xyz=0.00799999999999995 0 -0.123 rpy=0 0 0 -> xyz=0.007 0 -0.128 rpy=0 0 0
- joint right_arm5: limit lower=-1.57079633 upper=1.57079633 effort=0 velocity=0 -> lower=0 upper=0 effort=0 velocity=0; origin xyz=-0.0135999999999992 0 -0.1 rpy=0 0 0 -> xyz=-0.0146 0 -0.1 rpy=0 0 0
- joint right_arm6: limit lower=-1.57079633 upper=1.57079633 effort=0 velocity=0 -> lower=0 upper=0 effort=0 velocity=0; origin xyz=0.00548999599679659 0 -0.113357392395326 rpy=0 0 0 -> xyz=0.005 0 -0.12136 rpy=0 0 0
- joint right_arm7: limit lower=-1.57079633 upper=1.57079633 effort=0 velocity=0 -> lower=0 upper=0 effort=0 velocity=0; origin xyz=-0.0154170897275939 -0.0182000000001118 -0.0583391608133426 rpy=0 0 0 -> xyz=-0.0145 -0.02765 -0.05999 rpy=0 0 0
- joint right_arm8: axis -1 0 0 -> 1 0 0; limit lower=-1.57079633 upper=0.00000000 effort=0 velocity=0 -> lower=0 upper=0 effort=0 velocity=0; origin xyz=0.0182000000001126 0.00245122024342487 -0.0373617039078002 rpy=0 0 0 -> xyz=-0.0171 0.023417 -0.065349 rpy=0 0 0
- joint waist_Link: limit lower=-1.57079633 upper=1.57079633 effort=0 velocity=0 -> lower=0 upper=0 effort=0 velocity=0; origin xyz=0.00189999999999996 -0.098 0.0435000000000001 rpy=0 0 0 -> xyz=0 0 0.04 rpy=0 0 0
- joint whel_Link1: origin xyz=0.201 -0.465 -0.0349999999999996 rpy=0 0 0 -> xyz=0.201 -0.465 -0.035 rpy=0 0 0
- joint whel_Link2: origin xyz=-0.201 -0.465 -0.0349999999999996 rpy=0 0 0 -> xyz=-0.201 -0.465 -0.035 rpy=0 0 0
- joint whel_Link3: origin xyz=-0.201 -0.015 -0.0349999999999999 rpy=0 0 0 -> xyz=-0.201 -0.015 -0.035 rpy=0 0 0

Commit message: mark

File: URDF/aider/urdf/aider_pro.SLDASM.urdf (robot description, URDF)
Before this commit: robot aider_pro.SLDASM, 27 links, 26 joints
Joints:
- joint left_arm2: axis 0 1 0 -> 0 -1 0
- joint left_arm3: axis 0 0 1 -> 0 0 -1
- joint left_arm4: axis 1 0 0 -> -1 0 0
- joint left_arm5: axis 0 0 1 -> 0 0 -1
- joint left_arm6: axis 1 0 0 -> -1 0 0
- joint left_arm7: axis 0 1 0 -> 0 -1 0
- joint left_arm8: axis 1 0 0 -> -1 0 0
- joint right_arm8: axis 1 0 0 -> -1 0 0

Commit message: 新版URDF

File: URDF/aider/urdf/aider_pro.SLDASM.urdf (robot description, URDF)
Before this commit: robot aider_pro.SLDASM, 27 links, 26 joints
Links:
- link head_Link: mass 0.0401514926582811 -> 0.0401514926582812
- link left_arm8: mass 0.0398761874096987 -> 0.0398761874096988
- link left_hand_tcp: mass 0.000144 -> 0.000143995915056227
- link right_arm1: mass 0.27717 -> 0.277168822184387
- link right_arm3: mass 0.16242 -> 0.162415092593513
- link right_arm5: mass 0.050386 -> 0.0503857005011349
- link right_arm6: mass 0.047198 -> 0.0471983447304541
- link right_arm8: mass 0.039876 -> 0.0398758267789968
- link right_hand_tcp: mass 0.000144 -> 0.000143995915056229
- link whel_Link4: mass None -> 0.286092750982275
Joints:
- joint head_Link: limit lower=0 upper=0 effort=0 velocity=0 -> lower=-1.04719755 upper=1.04719755 effort=0 velocity=0
- joint head_Link2: limit lower=0 upper=0 effort=0 velocity=0 -> lower=-0.52359878 upper=0.78539816 effort=0 velocity=0
- joint left_arm1: limit lower=0 upper=0 effort=0 velocity=0 -> lower=-2.35619449 upper=2.35619449 effort=0 velocity=0
- joint left_arm2: limit lower=0 upper=0 effort=0 velocity=0 -> lower=-2.61799388 upper=1.57079633 effort=0 velocity=0
- joint left_arm3: limit lower=0 upper=0 effort=0 velocity=0 -> lower=-1.57079633 upper=1.57079633 effort=0 velocity=0
- joint left_arm4: limit lower=0 upper=0 effort=0 velocity=0 -> lower=0.00000000 upper=2.35619449 effort=0 velocity=0; origin xyz=-0.0244 0 -0.115 rpy=0 0 0 -> xyz=-0.0244000000000001 0 -0.115 rpy=0 0 0
- joint left_arm5: limit lower=0 upper=0 effort=0 velocity=0 -> lower=-1.57079633 upper=1.57079633 effort=0 velocity=0
- joint left_arm6: limit lower=0 upper=0 effort=0 velocity=0 -> lower=-1.57079633 upper=1.57079633 effort=0 velocity=0; origin xyz=-0.018 0 -0.10136 rpy=0 0 0 -> xyz=-0.018 0 -0.101357392395326 rpy=0 0 0
- joint left_arm7: limit lower=0 upper=0 effort=0 velocity=0 -> lower=-1.57079633 upper=1.57079633 effort=0 velocity=0; origin xyz=0.0275 -0.02965 -0.05999 rpy=0 0 0 -> xyz=0.0275 -0.0296499999999485 -0.0599903810567667 rpy=0 0 0
- joint left_arm8: limit lower=0 upper=0 effort=0 velocity=0 -> lower=-1.57079633 upper=0.00000000 effort=0 velocity=0; origin xyz=0.028543 0.025417 -0.065349 rpy=0 0 0 -> xyz=0.0285425250176359 0.0254170897275924 -0.0653487797565745 rpy=0 0 0
- joint left_hand_tcp: origin xyz=-0.0285425250176357 0.12828023583548 -0.0210756042379271 rpy=0 0 0 -> xyz=0 0.153697325563072 -0.0864243839945016 rpy=0 0 0; parent left_arm8 -> left_arm7
- joint lift_Link: limit lower=0 upper=0 effort=0 velocity=0 -> lower=0.00000000 upper=0.50000000 effort=0 velocity=0
- joint right_arm1: limit lower=0 upper=0 effort=0 velocity=0 -> lower=-2.35619449 upper=2.35619449 effort=0 velocity=0
- joint right_arm2: limit lower=0 upper=0 effort=0 velocity=0 -> lower=-2.61799388 upper=1.57079633 effort=0 velocity=0
- joint right_arm3: limit lower=0 upper=0 effort=0 velocity=0 -> lower=-1.57079633 upper=1.57079633 effort=0 velocity=0
- joint right_arm4: limit lower=0 upper=0 effort=0 velocity=0 -> lower=-2.35619449 upper=0.00000000 effort=0 velocity=0; origin xyz=0.007 0 -0.128 rpy=0 0 0 -> xyz=0.00699999999999987 0 -0.128 rpy=0 0 0
- joint right_arm5: limit lower=0 upper=0 effort=0 velocity=0 -> lower=-1.57079633 upper=1.57079633 effort=0 velocity=0
- joint right_arm6: limit lower=0 upper=0 effort=0 velocity=0 -> lower=-1.57079633 upper=1.57079633 effort=0 velocity=0; origin xyz=0.005 0 -0.12136 rpy=0 0 0 -> xyz=0.00499999999999995 0 -0.121357392395326 rpy=0 0 0
- joint right_arm7: limit lower=0 upper=0 effort=0 velocity=0 -> lower=-1.57079633 upper=1.57079633 effort=0 velocity=0; origin xyz=-0.0145 -0.02765 -0.05999 rpy=0 0 0 -> xyz=-0.0145000000000001 -0.0276499999999477 -0.0599903810567671 rpy=0 0 0
- joint right_arm8: limit lower=0 upper=0 effort=0 velocity=0 -> lower=-1.57079633 upper=0.00000000 effort=0 velocity=0; origin xyz=-0.0171 0.023417 -0.065349 rpy=0 0 0 -> xyz=-0.0171 0.0234170897275935 -0.0653487797565743 rpy=0 0 0
- joint right_hand_tcp: origin xyz=0.0171000000000001 0.12828023583548 -0.0210756042379271 rpy=0 0 0 -> xyz=0 0.151697325563073 -0.0864243839945014 rpy=0 0 0; parent right_arm8 -> right_arm7
- joint waist_Link: limit lower=0 upper=0 effort=0 velocity=0 -> lower=-1.57079633 upper=1.57079633 effort=0 velocity=0
- joint whel_Link1: origin xyz=0.201 -0.465 -0.035 rpy=0 0 0 -> xyz=0.201 -0.465 -0.0349999999999996 rpy=0 0 0
- joint whel_Link2: origin xyz=-0.201 -0.465 -0.035 rpy=0 0 0 -> xyz=-0.201 -0.465 -0.0349999999999996 rpy=0 0 0
- joint whel_Link3: origin xyz=-0.201 -0.015 -0.035 rpy=0 0 0 -> xyz=-0.201 -0.015 -0.0349999999999999 rpy=0 0 0
