Commit message: fix: 修复仿真显示 - URDF改名+TCP紫色球+mesh压缩产物

File: URDF/aider/urdf/aider_pro.SLDASM.urdf (robot description, URDF)
Before this commit: robot aider_pro.SLDASM, 27 links, 26 joints
Links:
- removed link left_hand_tcp
- removed link right_hand_tcp
- added link left_TCP, mass 0.523598775598299; collision sphere radius=0.02; visual sphere radius=0.02
- added link left_arm12, mass 0.0232107216134867; collision mesh filename=package://aider_pro01/meshes/left_arm12.STL; visual mesh filename=package://aider_pro01/meshes/left_arm12.STL
- added link right_TCP, mass 0.523598775598299; collision sphere radius=0.02; visual sphere radius=0.02
- added link right_arm12, mass 0.0232107216134868; collision mesh filename=package://aider_pro01/meshes/right_arm12.STL; visual mesh filename=package://aider_pro01/meshes/right_arm12.STL
- link base_link: mass 1.8672299751897 -> 10.4066594647559; geometry collision mesh filename=package://aider_pro01/meshes/base_link.STL; visual mesh filename=package://aider_pro01/meshes/base_link.STL
- link head_Link: mass 0.0401514926582812 -> 0.0675121095939233; geometry collision mesh filename=package://aider_pro01/meshes/head_Link.STL; visual mesh filename=package://aider_pro01/meshes/head_Link.STL
- link head_Link2: mass 0.189625426643452 -> 0.00790145083618025; geometry collision mesh filename=package://aider_pro01/meshes/head_Link2.STL; visual mesh filename=package://aider_pro01/meshes/head_Link2.STL
- link left_arm1: mass 0.2771689234867 -> 0.285085172303553; geometry collision mesh filename=package://aider_pro01/meshes/left_arm1.STL; visual mesh filename=package://aider_pro01/meshes/left_arm1.STL
- link left_arm2: mass 0.173551520246761 -> 0.173551481358342; geometry collision mesh filename=package://aider_pro01/meshes/left_arm2.STL; visual mesh filename=package://aider_pro01/meshes/left_arm2.STL
- link left_arm3: mass 0.162415224100578 -> 0.16242378611503; geometry collision mesh filename=package://aider_pro01/meshes/left_arm3.STL; visual mesh filename=package://aider_pro01/meshes/left_arm3.STL
- link left_arm4: mass 0.061262551263452 -> 0.162938668455009; geometry collision mesh filename=package://aider_pro01/meshes/left_arm4.STL; visual mesh filename=package://aider_pro01/meshes/left_arm4.STL
- link left_arm5: mass 0.0503857298730898 -> 0.273974650527036; geometry collision mesh filename=package://aider_pro01/meshes/left_arm5.STL; visual mesh filename=package://aider_pro01/meshes/left_arm5.STL
- link left_arm6: mass 0.0471985933288053 -> 0.296122979657166; geometry collision mesh filename=package://aider_pro01/meshes/left_arm6.STL; visual mesh filename=package://aider_pro01/meshes/left_arm6.STL
- link left_arm7: mass 0.103857648360567 -> 0.127525300289075; geometry collision mesh filename=package://aider_pro01/meshes/left_arm7.STL; visual mesh filename=package://aider_pro01/meshes/left_arm7.STL
- link left_arm8: mass 0.0398761874096988 -> 0.0232107216134867; geometry collision mesh filename=package://aider_pro01/meshes/left_arm8.STL; visual mesh filename=package://aider_pro01/meshes/left_arm8.STL
- link lift_Link: mass 0.590735662767956 -> 0.494039474476232; geometry collision mesh filename=package://aider_pro01/meshes/lift_Link.STL; visual mesh filename=package://aider_pro01/meshes/lift_Link.STL
- link right_arm1: mass 0.277168822184387 -> 0.285085172303553; geometry collision mesh filename=package://aider_pro01/meshes/right_arm1.STL; visual mesh filename=package://aider_pro01/meshes/right_arm1.STL
- link right_arm2: mass 0.210693834825324 -> 0.173551481358041; geometry collision mesh filename=package://aider_pro01/meshes/right_arm2.STL; visual mesh filename=package://aider_pro01/meshes/right_arm2.STL
- link right_arm3: mass 0.162415092593513 -> 0.158058522783778; geometry collision mesh filename=package://aider_pro01/meshes/right_arm3.STL; visual mesh filename=package://aider_pro01/meshes/right_arm3.STL
- link right_arm4: mass 0.0612625148219103 -> 0.162938667719021; geometry collision mesh filename=package://aider_pro01/meshes/right_arm4.STL; visual mesh filename=package://aider_pro01/meshes/right_arm4.STL
- link right_arm5: mass 0.0503857005011349 -> 0.262060771333877; geometry collision mesh filename=package://aider_pro01/meshes/right_arm5.STL; visual mesh filename=package://aider_pro01/meshes/right_arm5.STL
- link right_arm6: mass 0.0471983447304541 -> 0.296122979657166; geometry collision mesh filename=package://aider_pro01/meshes/right_arm6.STL; visual mesh filename=package://aider_pro01/meshes/right_arm6.STL
- link right_arm7: mass 0.103857535053998 -> 0.127525310280888; geometry collision mesh filename=package://aider_pro01/meshes/right_arm7.STL; visual mesh filename=package://aider_pro01/meshes/right_arm7.STL
- link right_arm8: mass 0.0398758267789968 -> 0.0232107216134868; geometry collision mesh filename=package://aider_pro01/meshes/right_arm8.STL; visual mesh filename=package://aider_pro01/meshes/right_arm8.STL
- link waist_Link: mass 1.90391027149609 -> 0.862993792172381; geometry collision mesh filename=package://aider_pro01/meshes/waist_Link.STL; visual mesh filename=package://aider_pro01/meshes/waist_Link.STL
- link whel_Link1: mass 0.286092916963456 -> 0.313871847085295; geometry collision mesh filename=package://aider_pro01/meshes/whel_Link1.STL; visual mesh filename=package://aider_pro01/meshes/whel_Link1.STL
- link whel_Link2: mass 0.286092750982276 -> 0.313871846832973; geometry collision mesh filename=package://aider_pro01/meshes/whel_Link2.STL; visual mesh filename=package://aider_pro01/meshes/whel_Link2.STL
- link whel_Link3: mass 0.286092916963456 -> 0.313871847243845; geometry collision mesh filename=package://aider_pro01/meshes/whel_Link3.STL; visual mesh filename=package://aider_pro01/meshes/whel_Link3.STL
- link whel_Link4: mass 0.286092750982275 -> 0.313871845736711; geometry collision mesh filename=package://aider_pro01/meshes/whel_Link4.STL; visual mesh filename=package://aider_pro01/meshes/whel_Link4.STL
Joints:
- removed joint left_hand_tcp
- removed joint right_hand_tcp
- added joint left_TCP: type fixed, parent left_arm7, child left_TCP, origin xyz=0 -0.24221 0.026 rpy=0 0 0, axis 0 0 0, limit lower=0 upper=0 effort=0 velocity=0
- added joint left_arm12: type revolute, parent left_arm7, child left_arm12, origin xyz=-0.0200596230640996 -0.141 0.0358036484876377 rpy=0 1.43116998667327 0, axis 0 0 -1, limit lower=0 upper=0 effort=0 velocity=0
- added joint right_TCP: type fixed, parent right_arm7, child right_TCP, origin xyz=0.0035364 -0.24218 0.026 rpy=1.5562 1.5708 0, axis 0 0 0, limit lower=0 upper=0 effort=0 velocity=0
- added joint right_arm12: type revolute, parent right_arm7, child right_arm12, origin xyz=0.0221161621566623 -0.140692088784192 0.0161963515032877 rpy=-3.12713369251084 -1.43115529453554 -3.14159265358958, axis 0 0 -1, limit lower=0 upper=0 effort=0 velocity=0
- joint head_Link: limit lower=-1.04719755 upper=1.04719755 effort=0 velocity=0 -> lower=0 upper=0 effort=0 velocity=0; origin xyz=0 -0.163916235400507 0.448200000000012 rpy=0 0 0 -> xyz=0 0.322 0 rpy=1.5707963267949 1.5707963267949 0
- joint head_Link2: axis 1 0 0 -> 0 0 -1; limit lower=-0.52359878 upper=0.78539816 effort=0 velocity=0 -> lower=0 upper=0 effort=0 velocity=0; origin xyz=-0.0183049377506555 -0.0130000000000431 0.0225999999999615 rpy=0 0 0 -> xyz=0 0 -0.0369999999999999 rpy=-1.5707963267949 0 1.5707963267949
- joint left_arm1: axis 1 0 0 -> 0 0 -1; limit lower=-2.35619449 upper=2.35619449 effort=0 velocity=0 -> lower=0 upper=0 effort=0 velocity=0; origin xyz=0.105510000000001 -0.148985915842714 0.3225 rpy=0 0 0 -> xyz=0 0.195000000000003 0.0885099999999956 rpy=-3.14159265358979 0 3.14159265358979
- joint left_arm2: axis 0 -1 0 -> 0 0 -1; limit lower=-2.61799388 upper=1.57079633 effort=0 velocity=0 -> lower=0 upper=0 effort=0 velocity=0; origin xyz=0.0420000000000001 -0.0399999999999999 0 rpy=0 0 0 -> xyz=0.0289999999999984 0 -0.0569999999999984 rpy=3.14159265358979 1.5707963267949 0
- joint left_arm3: limit lower=-1.57079633 upper=1.57079633 effort=0 velocity=0 -> lower=0 upper=0 effort=0 velocity=0; origin xyz=0 0.0399999806952274 -0.133399999999999 rpy=0 0 0 -> xyz=0 0.125399999999998 0.0289999806952269 rpy=1.57079632679488 0 3.14159265358979
- joint left_arm4: axis -1 0 0 -> 0 0 -1; limit lower=0.00000000 upper=2.35619449 effort=0 velocity=0 -> lower=0 upper=0 effort=0 velocity=0; origin xyz=-0.0244000000000001 0 -0.115 rpy=0 0 0 -> xyz=0.0163999999999997 -1.8212984132765E-05 0.122999999999998 rpy=-1.5707963267949 0 1.57079632679489
- joint left_arm5: axis 0 0 -1 -> 0 0 1; limit lower=-1.57079633 upper=1.57079633 effort=0 velocity=0 -> lower=0 upper=0 effort=0 velocity=0; origin xyz=0.032 0 -0.12 rpy=0 0 0 -> xyz=-0.00146589510149292 -0.100389297993122 0.0289999999999995 rpy=1.58539739441215 -1.5707963267949 0
- joint left_arm6: axis -1 0 0 -> 0 0 -1; limit lower=-1.57079633 upper=1.57079633 effort=0 velocity=0 -> lower=0 upper=0 effort=0 velocity=0; origin xyz=-0.018 0 -0.101357392395326 rpy=0 0 0 -> xyz=0 -0.00550000000001608 0.121999999999962 rpy=-1.5707963267949 0 -3.14159265358979
- joint left_arm7: axis 0 -1 0 -> 0 0 -1; limit lower=-1.57079633 upper=1.57079633 effort=0 velocity=0 -> lower=0 upper=0 effort=0 velocity=0; origin xyz=0.0275 -0.0296499999999485 -0.0599903810567667 rpy=0 0 0 -> xyz=0.0259000000000001 0 0 rpy=-1.57079632679492 -1.55619525917765 1.57079632679492
- joint left_arm8: axis -1 0 0 -> 0 0 -1; limit lower=-1.57079633 upper=0.00000000 effort=0 velocity=0 -> lower=0 upper=0 effort=0 velocity=0; origin xyz=0.0285425250176359 0.0254170897275924 -0.0653487797565745 rpy=0 0 0 -> xyz=-0.0165802955410368 -0.141 0.0110469467689665 rpy=3.14159265358979 -1.43116998667327 -3.14159265358979
- joint lift_Link: axis 0 0 1 -> 0 0 -1; limit lower=0.00000000 upper=0.50000000 effort=0 velocity=0 -> lower=0 upper=0 effort=0 velocity=0; origin xyz=0 -0.0930000000000004 0.577289106240448 rpy=0 0 0 -> xyz=0 -0.0929999999999999 0.637959988593697 rpy=0 0 0
- joint right_arm1: axis -1 0 0 -> 0 0 -1; limit lower=-2.35619449 upper=2.35619449 effort=0 velocity=0 -> lower=0 upper=0 effort=0 velocity=0; origin xyz=-0.0650100000000005 -0.14898591584271 0.322499999999999 rpy=0 0 0 -> xyz=1.40841572922046E-05 0.194999999999996 -0.088509999999995 rpy=0 0 0
- joint right_arm2: axis 0 -1 0 -> 0 0 -1; limit lower=-2.61799388 upper=1.57079633 effort=0 velocity=0 -> lower=0 upper=0 effort=0 velocity=0; origin xyz=-0.0825 -0.0205 0 rpy=0 0 0 -> xyz=-0.0289999999999998 0 -0.057 rpy=0 1.5707963267949 0
- joint right_arm3: limit lower=-1.57079633 upper=1.57079633 effort=0 velocity=0 -> lower=0 upper=0 effort=0 velocity=0; origin xyz=0 0.0204999806952246 -0.1204 rpy=0 0 0 -> xyz=0 -0.1254 0.0289999806953687 rpy=-1.57079632679488 0 -3.14159265358979
- joint right_arm4: axis 1 0 0 -> 0 0 -1; limit lower=-2.35619449 upper=0.00000000 effort=0 velocity=0 -> lower=0 upper=0 effort=0 velocity=0; origin xyz=0.00699999999999987 0 -0.128 rpy=0 0 0 -> xyz=0.0163999999999998 0 0.122999999999991 rpy=1.57079632679485 0 -1.5707963267949
- joint right_arm5: limit lower=-1.57079633 upper=1.57079633 effort=0 velocity=0 -> lower=0 upper=0 effort=0 velocity=0; origin xyz=-0.0146 0 -0.1 rpy=0 0 0 -> xyz=-0.00146589510162229 0.10038929799312 0.0289999999998398 rpy=1.55619525917765 -1.5707963267949 0
- joint right_arm6: axis 1 0 0 -> 0 0 -1; limit lower=-1.57079633 upper=1.57079633 effort=0 velocity=0 -> lower=0 upper=0 effort=0 velocity=0; origin xyz=0.00499999999999995 0 -0.121357392395326 rpy=0 0 0 -> xyz=0 -0.00550000000000189 -0.121999999999996 rpy=1.57079632679491 0 0
- joint right_arm7: axis 0 -1 0 -> 0 0 -1; limit lower=-1.57079633 upper=1.57079633 effort=0 velocity=0 -> lower=0 upper=0 effort=0 velocity=0; origin xyz=-0.0145000000000001 -0.0276499999999477 -0.0599903810567671 rpy=0 0 0 -> xyz=-0.0258999999999558 0 0 rpy=-1.57079632679505 1.55619525917764 -1.57079632679502
- joint right_arm8: axis -1 0 0 -> 0 0 -1; limit lower=-1.57079633 upper=0.00000000 effort=0 velocity=0 -> lower=0 upper=0 effort=0 velocity=0; origin xyz=-0.0171 0.0234170897275935 -0.0653487797565743 rpy=0 0 0 -> xyz=0.0186372055079729 -0.140742888875552 0.040953053221959 rpy=-0.0144589610789541 1.43115529453554 0
- joint waist_Link: axis -1 0 0 -> 0 0 -1; limit lower=-1.57079633 upper=1.57079633 effort=0 velocity=0 -> lower=0 upper=0 effort=0 velocity=0; origin xyz=0 0 0.04 rpy=0 0 0 -> xyz=0 -0.149 0.0975000000000001 rpy=1.5707963267949 0 1.5707963267949
- joint whel_Link1: axis -1 0 0 -> 0 0 -1; origin xyz=0.201 -0.465 -0.0349999999999996 rpy=0 0 0 -> xyz=0.176 -0.465 -0.035 rpy=1.5708 0 1.5708
- joint whel_Link2: axis 1 0 0 -> 0 0 -1; origin xyz=-0.201 -0.465 -0.0349999999999996 rpy=0 0 0 -> xyz=-0.176 -0.465 -0.035 rpy=1.5708 0 -1.5708
- joint whel_Link3: axis 1 0 0 -> 0 0 -1; origin xyz=-0.201 -0.015 -0.0349999999999999 rpy=0 0 0 -> xyz=0.176 -0.015 -0.035 rpy=1.5708 0 1.5708
- joint whel_Link4: axis -1 0 0 -> 0 0 -1; origin xyz=0.201 -0.015 -0.0349999999999999 rpy=0 0 0 -> xyz=-0.176 -0.015 -0.0349999999999989 rpy=1.5707963267949 0 -1.5707963267949

Commit message: fix(vr): 手腕俯仰/偏航方向修复 + 位置映射X恢复
- vr_handler: 去掉 wrist_flex/yaw 多余负号(翻滚双重负号抵消一直正确)
- utils: 位置映射 X 恢复 -x(配合真机 arm1-4 direction=-1 镜像)
- URDF: 修正左右手腕关节轴方向
- recorder: 录制增加 VR 手柄 position 字段

File: URDF/aider/urdf/aider_pro.SLDASM.urdf (robot description, URDF)
Before this commit: robot aider_pro01, 29 links, 28 joints
Joints:
- joint left_arm5: axis 0 0 1 -> 0.000000 -0.014601 -0.999893
- joint left_arm6: axis 0 0 -1 -> 1.000000 0.000000 0.000000
- joint left_arm7: axis 0 0 -1 -> -0.999574 0.029198 -0.000000
- joint right_arm5: axis 0 0 -1 -> -0.000000 -0.014601 0.999893
- joint right_arm6: axis 0 0 -1 -> 1.000000 0.000000 0.000000
- joint right_arm7: axis 0 0 -1 -> 0.999574 0.029198 0.000000
